Commit message: CHG: remove namespace lio_sam
instead of using namespace lidar_undistortion_3d.

File: lidar_undistortion_3d/launch/include/config/robot.urdf.xacro (robot description, xacro)
@@ -15,8 +15,8 @@
     <origin xyz="0 0 0" rpy="0 0 0" />
   </joint>
-  <link name="velodyne"> </link>
-  <joint name="velodyne_joint" type="fixed">
+  <link name="laser_link"> </link>
+  <joint name="laser_joint" type="fixed">
     <parent link="chassis_link" />
-    <child link="velodyne" />
+    <child link="laser_link" />
     <origin xyz="0 0 0" rpy="0 0 0" />
   </joint>
